Commit message: clean the enviroment and then ready for the deployment remove the issue of missing robot in simulation. add the feature of computer vision

File: src/clearpath_common/clearpath_platform_description/urdf/generic/gazebo.urdf.xacro (robot description, xacro)
@@ -3,9 +3,12 @@
   <xacro:if value="$(arg is_sim)">
     <gazebo>
-      <plugin filename="libgz_ros2_control-system.so" name="gz_ros2_control::GazeboSimROS2ControlPlugin">
+      <plugin filename="libign_ros2_control-system.so" name="ign_ros2_control::IgnitionROS2ControlPlugin">
         <parameters>$(arg gazebo_controllers)</parameters>
+        <robot_param>robot_description</robot_param>
+        <robot_param_node>robot_state_publisher</robot_param_node>
         <ros>
           <remapping>~/odom:=platform/odom</remapping>
           <remapping>~/cmd_vel:=platform/cmd_vel</remapping>
+          <remapping>~/cmd_vel_unstamped:=platform/cmd_vel</remapping>
           <remapping>/tf:=tf</remapping>
           <remapping>/tf_static:=tf_static</remapping>
@@ -20,5 +23,5 @@
     </gazebo>
     <gazebo>
-      <plugin filename="libgz-sim-pose-publisher-system.so" name="gz::sim::systems::PosePublisher">
+      <plugin filename="libignition-gazebo-pose-publisher-system.so" name="ignition::gazebo::systems::PosePublisher">
         <publish_link_pose>true</publish_link_pose>
         <publish_nested_model_pose>true</publish_nested_model_pose>

File: src/clearpath_common/clearpath_platform_description/urdf/j100/j100.urdf.xacro (robot description, xacro)
@@ -51,5 +51,5 @@
     <!-- Hardware  -->
     <xacro:if value="$(arg is_sim)">
-      <xacro:property name="hardware_plugin" value="gz_ros2_control/GazeboSimSystem"/>
+      <xacro:property name="hardware_plugin" value="ign_ros2_control/IgnitionSystem"/>
     </xacro:if>
     <xacro:unless value="$(arg is_sim)">
